File: Battery/Battery.sch (KiCad schematic (older format))
At the start: 1 part

Commit message: Batteriju izklājlaukumu mājasdarbs
Parts:
- BT1: footprint Battery_Holder:S8211-46R -> Battery_Holder:S8401-46
Changed lines of the file:
@@
 F 0 "BT1" H 1828 2836 50  0000 L CNN
 F 1 "Battery_Cell" H 1828 2745 50  0000 L CNN
-F 2 "Battery_Holder:S8211-46R" V 1710 2800 50  0001 C CNN
+F 2 "Battery_Holder:S8401-46" V 1710 2800 50  0001 C CNN
 F 3 "https://pdf1.alldatasheet.com/datasheet-pdf/view/563073/HARWIN/S8211-46R.html" V 1710 2800 50  0001 C CNN
 	1    1710 2740
