File: Single_transistor_AMP/Single_transistor_AMP.kicad_pcb (KiCad board)
At the start: 2 copper layers, 22 parts, among them J1 AudioJack2_Ground, J2 12V, J3 Signal out, Q1 BC546, Q2 BC546, Q3 BD139

Commit message: Treniņuzdevumi
Parts:
- removed C3: 10uF, Capacitor_SMD:CP_Elec_4x4.5
- removed C4: 3.3uF, Capacitor_SMD:CP_Elec_4x4.5
- removed Q2: BC546, Package_TO_SOT_THT:TO-92
- removed R10, R9: 120, Resistor_SMD:R_0402_1005Metric
- removed R6: 56k, Resistor_SMD:R_0402_1005Metric
- removed R7: 6k8, Resistor_SMD:R_0402_1005Metric
- removed R8: 2k7, Resistor_SMD:R_0402_1005Metric
- C2: value 3.3uF -> 470uF
- C5: value 22uF -> 470uF
- J2: value 12V -> 32V; footprint Connector:Banana_Jack_2Pin -> Connector:JWT_A3963_1x02_P3.96mm_Vertical
- J3: footprint Connector:Banana_Jack_2Pin -> Connector:JWT_A3963_1x02_P3.96mm_Vertical
- Q3: value BD139 -> TIP140; footprint Package_TO_SOT_THT:TO-126-3_Vertical -> Package_TO_SOT_THT:TO-247-3_Vertical
- R1: value 56k -> 110k; footprint Resistor_SMD:R_0402_1005Metric -> Resistor_SMD:R_0603_1608Metric
- R11: value 47,5 -> 16; footprint Resistor_SMD:R_0402_1005Metric -> Resistor_SMD:R_0603_1608Metric
- R2: footprint Resistor_SMD:R_0402_1005Metric -> Resistor_SMD:R_0603_1608Metric
- R3: value 2k7 -> 3k; footprint Resistor_SMD:R_0402_1005Metric -> Resistor_SMD:R_0603_1608Metric
- R4, R5: value 120 -> 100; footprint Resistor_SMD:R_0402_1005Metric -> Resistor_SMD:R_0603_1608Metric
- moved J1 99.5 mm to (211.6, 159.5), turned to 90 degrees
- moved Q3 87.1 mm to (227.6, 158.2), turned to 90 degrees
- moved J2 83.2 mm to (209.4, 143.4), turned to 90 degrees
- moved J3 80.2 mm to (209.4, 152.3), turned to 90 degrees
- moved C5 75.5 mm to (217.9, 152.4)
- moved R11 67.1 mm to (219.3, 144.3), turned to 180 degrees
- moved Q1 62.5 mm to (217.6, 141.5)
- moved C2 60.5 mm to (217.8, 147.4), turned to 180 degrees
- moved R5 60.2 mm to (216.0, 144.3), turned to 180 degrees
- moved R2 59.4 mm to (215.3, 142.0), turned to 270 degrees
- moved C1 59.0 mm to (224.0, 141.1), turned to 90 degrees
- moved R4 57.8 mm to (220.6, 137.9)
- moved R1 56.8 mm to (215.3, 138.9), turned to 270 degrees
- moved R3 55.0 mm to (217.6, 137.9)
Connections:
- Q1 pad 2: Net-(C3-Pad1) -> Net-(Q1-Pad2)
- Q3 pad 1: Net-(Q2-Pad2) -> Net-(Q1-Pad2)
- R3 pad 2: Net-(C3-Pad1) -> Net-(Q1-Pad2)
Routing:
- net Net-(J2-Pad1): track 0.00 -> 34.6 mm, vias 0 -> 2
- net Net-(Q1-Pad2): track 0.00 -> 25.5 mm
- net Net-(C1-Pad1): track 0.00 -> 25.4 mm, vias 0 -> 2
- net Net-(C5-Pad1): track 0.00 -> 22.7 mm
- net Net-(C2-Pad1): track 0.00 -> 14.1 mm, vias 0 -> 2
- net Net-(C1-Pad2): track 0.00 -> 12.6 mm
- net Net-(C5-Pad2): track 0.00 -> 11.3 mm
- net Net-(Q1-Pad3): track 0.00 -> 3.67 mm
- added copper zone on B.Cu, net (none)
- added copper zone on F.Cu, net (none)
- added copper zone on B.Cu, net GND
- added copper zone on F.Cu, net GND
Other:
- board outline added: 24.9 x 27.3 mm
- net class POWER added: clearance 0.2, trace_width 0.3, via_dia 0.8, via_drill 0.4
- net class SIGNAL added: clearance 0.2, trace_width 0.2, via_dia 0.8, via_drill 0.4

Commit message: Izpildīts 8 lekcijas MD
Parts:
- moved Q3 132.8 mm to (103.1, 111.9), turned to 0 degrees
- moved J1 112.7 mm to (102.6, 130.7)
- moved R3 112.2 mm to (107.6, 116.0)
- moved C1 111.1 mm to (114.3, 123.4), turned to 180 degrees
- moved Q1 108.1 mm to (111.9, 118.9), turned to 90 degrees
- moved J2 107.7 mm to (103.6, 123.3)
- moved R11 107.5 mm to (115.6, 116.2), turned to 0 degrees
- moved R4 106.9 mm to (115.6, 118.1)
- moved R2 106.9 mm to (110.4, 121.5), turned to 180 degrees
- moved R1 105.8 mm to (110.4, 125.1), turned to 0 degrees
- moved C5 103.4 mm to (121.2, 116.1)
- moved R5 103.3 mm to (115.6, 120.0)
- moved C2 100.3 mm to (121.0, 120.9), turned to 0 degrees
- moved J3 89.3 mm to (122.6, 131.4), turned to 180 degrees
Routing:
- net Net-(J2-Pad1): track 34.6 -> 0.00 mm, vias 2 -> 0
- net Net-(Q1-Pad2): track 25.5 -> 0.00 mm
- net Net-(C1-Pad1): track 25.4 -> 0.00 mm, vias 2 -> 0
- net Net-(C5-Pad1): track 22.7 -> 0.00 mm
- net Net-(C2-Pad1): track 14.1 -> 0.00 mm, vias 2 -> 0
- net Net-(C1-Pad2): track 12.6 -> 0.00 mm
- net Net-(C5-Pad2): track 11.3 -> 0.00 mm
- net Net-(Q1-Pad3): track 3.67 -> 0.00 mm
- removed copper zone on B.Cu, net (none)
- removed copper zone on F.Cu, net (none)
- removed copper zone on B.Cu, net GND
- removed copper zone on F.Cu, net GND
Other:
- board size 24.9 x 27.3 mm -> 25.2 x 26 mm
- net class POWER: clearance 0.2 -> 0.5
- board text added: "A-CLASS Amplifier Made by Rodrigo"

Commit message: 8 nodarbības MD
Parts:
- moved R1 3.81 mm to (110.2, 121.3)
- moved R2 3.69 mm to (110.2, 125.2)
- moved C2 2.41 mm to (121.0, 123.3)
- moved C5 2.41 mm to (121.2, 118.5)
- moved R3 1.03 mm to (106.6, 115.6)
- moved J2 0.58 mm to (103.6, 122.7)
- moved Q3 0.25 mm to (103.1, 111.6)
- moved C1 0.14 mm to (114.2, 123.3)
- turned R11 to 180 degrees
Connections:
- J2 pad 1: Net-(J2-Pad1) -> GND
- J2 pad 2: GND -> Net-(J2-Pad2)
- Q3 pad 2: Net-(J2-Pad1) -> Net-(J2-Pad2)
- R1 pad 1: Net-(J2-Pad1) -> Net-(J2-Pad2)
- R3 pad 1: Net-(J2-Pad1) -> Net-(J2-Pad2)
Routing:
- net Net-(C1-Pad1): track 0.00 -> 18.3 mm
- net Net-(J2-Pad2): track 0.00 -> 17.8 mm
- net Net-(C5-Pad2): track 0.00 -> 13.2 mm, vias 0 -> 2
- net Net-(Q1-Pad2): track 0.00 -> 9.97 mm, vias 0 -> 1
- net Net-(C5-Pad1): track 0.00 -> 9.49 mm
- net Net-(C1-Pad2): track 0.00 -> 7.88 mm
- net Net-(C2-Pad1): track 0.00 -> 6.40 mm
- net Net-(Q1-Pad3): track 0.00 -> 3.63 mm
- net GND: vias 0 -> 2
- added copper zone on F.Cu, net (none)
- added copper zone on B.Cu, net GND
- added copper zone on F.Cu, net GND
Other:
- net class POWER: clearance 0.5 -> 0.2; trace_width 0.3 -> 0.5
